File: MCM-iMX93-dev.kicad_pcb (KiCad board)
At the start: 4 copper layers, 78 x 79 mm, 46 parts, among them J1 USB_B_Mini, J10 Display, J11 External I2S, J12 RPi connector, J13 PTT, J6 GPIO, J7 USB boot, J8 UART, J9 5V supply, SW1 ON/OFF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

Commit message: started pcb routing
Parts:
- added REF**: LayerMarker_4_6.35x2.54mm_TextH1mm_P1.27mm, Symbol:LayerMarker_4_6.35x2.54mm_TextH1mm_P1.27mm, F.Cu at (115.3, 123.2)
- moved REF** 1.53 mm to (125.1, 88.9)
Routing:
- net /SPI1_MOSI: track 0.00 -> 75.4 mm, vias 0 -> 4
- net /~{LCD_CS}: track 0.00 -> 72.9 mm, vias 0 -> 4
- net /SPI1_SCK: track 0.00 -> 58.7 mm, vias 0 -> 4
- net /LCD_RS: track 0.00 -> 46.2 mm, vias 0 -> 2
- net GND: vias 57 -> 296
